File: outputs.kicad_sch (KiCad schematic)
At the start: 20 parts, among them J4 Conn_01x06, Q1 SSM3K318R, Q2 SSM3K318R, Q3 SSM3K318R, U8 BM2LC105, U9 BM2LC105

Commit message: Completed layout, slight changes to schematic to optimise routing, 12V proto supply rail removed
Parts:
- J4: footprint Connector_PinHeader_2.54mm:PinHeader_1x06_P2.54mm_Horizontal -> Connector_PinHeader_2.54mm:PinHeader_1x06_P2.54mm_Vertical
Changed lines of the file:
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@@
     (property "Reference" "J4" (id 0) (at 50.8 142.24 0))
     (property "Value" "Conn_01x06" (id 1) (at 50.8 144.78 0))
-    (property "Footprint" "Connector_PinHeader_2.54mm:PinHeader_1x06_P2.54mm_Horizontal" (id 2) (at 58.42 144.78 0)
+    (property "Footprint" "Connector_PinHeader_2.54mm:PinHeader_1x06_P2.54mm_Vertical" (id 2) (at 58.42 144.78 0)
       (effects (font (size 1.27 1.27)) hide)
     )
