File: perfectV2.1v0.kicad_pcb (KiCad board)
At the start: 2 copper layers, 140.5 x 100.3 mm, 170 parts, among them IC1 TEENSY_4.1, IC2 Trig Cond Socket, IC3 Trig Cond Socket, J1 Conn_02x20_Odd_Even, J2 Conn_01x02, J3 Conn_01x05, J4 Conn_01x05, J5 Conn_01x05, J6 Conn_01x03, J7 Conn_01x04, J8 Conn_01x06, Q1 SSM3K357R, Q2 SSM3K357R, Q3 SSM3K357R, U1 VNLD5090, U10 TC4424A, U11 TC4424A, U2 VNLD5090, U3 VNLD5090, U4 MPX4250, U5 LMV324LIDT, U6 SP720, U7 LM2940S-5.0/NOPB, U8 VNLD5090, U9 VNLD5090

Commit message: Removed previous PCB layout, updated title blocks, changed stackup
Parts:
- removed A1: Pololu_Breakout_DRV8825, Module:Pololu_Breakout-16_15.2x20.3mm
- removed C1, C25, C27: 0.01uF, Capacitor_SMD:C_0805_2012Metric
- removed C10, C11, C12, C17, C18, C20, C22, C23, C24, C26, C28, C3, C30, C4: 0.1uF, Capacitor_SMD:C_0805_2012Metric
- removed C13, C14, C15, C5, C6, C7: 0.22uF, Capacitor_SMD:C_0805_2012Metric
- removed C16: 10uF, Capacitor_Tantalum_SMD:CP_EIA-7343-31_Kemet-D
- removed C19: 22uF, Capacitor_SMD:C_0805_2012Metric_Pad1.15x1.40mm_HandSolder
- removed C2, C29, C31: 1uF, Capacitor_SMD:C_0805_2012Metric
- removed C21: 47uF, Capacitor_Tantalum_SMD:CP_EIA-3528-21_Kemet-B
- removed C8, C9: 470pf, Capacitor_SMD:C_0805_2012Metric
- removed D1, D19, D2, D20, D21, D22, D3, D7, D8: LED, LED_SMD:LED_0805_2012Metric
- removed D10, D15, D16, D17, D18, D4, D5, D6, D9: D, Diode_SMD:D_SOD-323
- removed D11, D12: D_Zener, Diode_SMD:D_SOD-323
- removed D13: B130-13-F, Diode_SMD:D_SMA
- removed D14: 1SMB5919BT3G, Diode_SMD:D_SMB
- removed F1, F2: Polyfuse, Fuse:Fuse_1812_4532Metric
- removed IC1: TEENSY_4.1, Teensy:Teensy41
- removed IC2, IC3: Trig Cond Socket, Package_DIP:DIP-8_W7.62mm_Socket
- removed J1: Conn_02x20_Odd_Even, Connector_IDC:IDC-Header_2x20_P2.54mm_Vertical
- removed J2: Conn_01x02, TerminalBlock_Phoenix:TerminalBlock_Phoenix_PT-1,5-2-5.0-H_1x02_P5.00mm_Horizontal
- removed J3, J4, J5: Conn_01x05, Connector_PinHeader_2.54mm:PinHeader_1x05_P2.54mm_Vertical
- removed J6: Conn_01x03, Connector_PinHeader_2.54mm:PinHeader_1x03_P2.54mm_Vertical
- removed J7: Conn_01x04, Connector_PinHeader_2.54mm:PinHeader_1x04_P2.54mm_Vertical
- removed J8: Conn_01x06, Connector_PinHeader_2.54mm:PinHeader_1x06_P2.54mm_Vertical
- removed JP1: Jumper_3_Bridged12, Jumper:SolderJumper-3_P1.3mm_Bridged12_RoundedPad1.0x1.5mm
- removed JP10, JP12, JP9: VR-HALL, Connector_PinHeader_2.54mm:PinHeader_1x03_P2.54mm_Vertical
- removed JP11, JP7, JP8: PULL-UP, Connector_PinHeader_2.54mm:PinHeader_1x02_P2.54mm_Vertical
- removed JP13: Ignition Voltage, Connector_PinHeader_2.54mm:PinHeader_1x03_P2.54mm_Vertical
- removed JP2, JP3, JP4, JP5, JP6: SolderJumper_2_Bridged, Jumper:SolderJumper-2_P1.3mm_Bridged_Pad1.0x1.5mm
- removed Q1, Q2, Q3: SSM3K357R, Package_TO_SOT_SMD:SOT-23
- removed R1, R10, R11, R2, R3, R42, R43, R49, R50, R59, R60, R67, R68: 100k, Resistor_SMD:R_0805_2012Metric
- removed R12, R13, R16, R25, R4, R41, R44, R45, R48, R5, R51, R52, R53, R54, R57, R6, R61, R62, R69, R70: 1k, Resistor_SMD:R_0805_2012Metric
- removed R14, R15, R20, R63, R64, R7, R71, R72, R8, R9: 2.4k, Resistor_SMD:R_0805_2012Metric
- removed R17: 3.9k, Resistor_SMD:R_0805_2012Metric
- removed R18, R19, R21, R22, R26, R27, R28, R39, R40: 470R, Resistor_SMD:R_0805_2012Metric
- removed R23, R24: 2.49k, Resistor_SMD:R_0805_2012Metric
- removed R29, R30, R33, R34: 180k, Resistor_SMD:R_0805_2012Metric
- removed R31, R32, R35, R36: 330k, Resistor_SMD:R_0805_2012Metric
- removed R37, R46: 10k, Resistor_SMD:R_0805_2012Metric
- removed R38: 120R, Resistor_SMD:R_0805_2012Metric
- removed R47: 2k, Resistor_SMD:R_0805_2012Metric
- removed R55, R56, R58: 220R, Resistor_SMD:R_0805_2012Metric
- removed R65, R66, R73, R74: 10R, Resistor_SMD:R_0805_2012Metric
- removed RV1: Varistor, Varistor:RV_Disc_D15.5mm_W4.7mm_P7.5mm
- removed S1: AYZ0202AGRLC, Misc:AYZ0202AGRLC
- removed U1, U2, U3, U8, U9: VNLD5090, Package_SO:SOIC-8_3.9x4.9mm_P1.27mm
- removed U10, U11: TC4424A, Package_SO:SOIC-8_3.9x4.9mm_P1.27mm
- removed U4: MPX4250, Misc:MPX4250
- removed U5: LMV324LIDT, Package_SO:SOIC-14_3.9x8.7mm_P1.27mm
- removed U6: SP720, Package_SO:SOIC-16_3.9x9.9mm_P1.27mm
- removed U7: LM2940S-5.0/NOPB, Package_TO_SOT_SMD:TO-263-3_TabPin2
Routing:
- net GND: track 910.1 -> 0.00 mm, vias 1 -> 0
- net 12V-SW: track 406.2 -> 0.00 mm, vias 2 -> 0
- net VDD: track 349.6 -> 0.00 mm, vias 1 -> 0
- net VDDA: track 223.3 -> 0.00 mm, vias 2 -> 0
- net BOOST-OUT: track 198.1 -> 0.00 mm, vias 1 -> 0
- net HC-1-OUT: track 195.6 -> 0.00 mm, vias 1 -> 0
- net ADC-Clamp-7: track 179.1 -> 0.00 mm, vias 3 -> 0
- net IDLE-OUT: track 175.5 -> 0.00 mm, vias 1 -> 0
- net ADC-Clamp-10: track 170.1 -> 0.00 mm, vias 3 -> 0
- net CRANK-IN: track 169.2 -> 0.00 mm, vias 1 -> 0
- net HC-2-OUT: track 164.5 -> 0.00 mm, vias 1 -> 0
- net ADC-Clamp-8: track 146.3 -> 0.00 mm, vias 1 -> 0
- net INJ-3-OUT: track 144.4 -> 0.00 mm, vias 1 -> 0
- net MAP-EXT: track 137.5 -> 0.00 mm, vias 3 -> 0
- net INJ-2-OUT: track 124.7 -> 0.00 mm, vias 1 -> 0
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- removed copper zone on B.Cu, net GND
- removed copper zone on F.Cu, net GND
Other:
- board outline removed
- copper layers 2 -> 4
- board text removed: "5V"
- board text removed: "BLUETOOTH"
- board text removed: "GND"
- board text removed: "MOUNT FLAT SIDE UP"
- board text removed: "PROTO CONNECTOR LINK"
- board text removed: "Prog"
- board text removed: "RX"
- board text removed: "Run"
- board text removed: "SEVER ASSOCIATED JUMPER WHEN USING PROTO CONNECTOR LINK"
- board text removed: "TX"

Commit message: Completed layout, slight changes to schematic to optimise routing, 12V proto supply rail removed
Parts:
- added A1: Pololu_Breakout_DRV8825, Module:Pololu_Breakout-16_15.2x20.3mm, F.Cu at (92.1, 131.2)
- added C1: 10uF, Capacitor_Tantalum_SMD:CP_EIA-7343-31_Kemet-D, F.Cu at (68.7, 82.0)
- added C10: 0.22uF, Capacitor_SMD:C_0805_2012Metric, F.Cu at (76.2, 161.6)
- added C11: 0.1uF, Capacitor_SMD:C_0805_2012Metric, F.Cu at (66.5, 165.1)
- added C12: 0.22uF, Capacitor_SMD:C_0805_2012Metric, F.Cu at (69.4, 166.1)
- added C13: 0.1uF, Capacitor_SMD:C_0805_2012Metric, F.Cu at (59.8, 161.0)
- added C14: 0.22uF, Capacitor_SMD:C_0805_2012Metric, F.Cu at (57.0, 162.0)
- added C15: 0.1uF, Capacitor_SMD:C_0805_2012Metric, F.Cu at (77.6, 137.2)
- added C16: 0.22uF, Capacitor_SMD:C_0805_2012Metric, F.Cu at (83.4, 137.2)
- added C17: 0.1uF, Capacitor_SMD:C_0805_2012Metric, F.Cu at (58.2, 156.1)
- added C18: 0.22uF, Capacitor_SMD:C_0805_2012Metric, F.Cu at (58.5, 158.9)
- added C19: 0.22uF, Capacitor_SMD:C_0805_2012Metric, F.Cu at (59.0, 141.2)
- added C2: 0.1uF, Capacitor_SMD:C_0805_2012Metric, F.Cu at (74.7, 79.3)
- added C20: 0.1uF, Capacitor_SMD:C_0805_2012Metric, F.Cu at (102.0, 160.9)
- added C21: 0.1uF, Capacitor_SMD:C_0805_2012Metric, F.Cu at (102.0, 164.5)
- added C22: 0.01uF, Capacitor_SMD:C_0805_2012Metric, F.Cu at (102.2, 151.0)
- added C23: 0.1uF, Capacitor_SMD:C_0805_2012Metric, F.Cu at (82.7, 121.4)
- added C24: 1uF, Capacitor_SMD:C_0805_2012Metric, F.Cu at (84.9, 121.5)
- added C25: 0.1uF, Capacitor_SMD:C_0805_2012Metric, F.Cu at (90.5, 121.5)
- added C26: 1uF, Capacitor_SMD:C_0805_2012Metric, F.Cu at (88.3, 121.5)
- added C27: 0.1uF, Capacitor_SMD:C_0805_2012Metric, F.Cu at (139.0, 114.0)
- added C28: 0.1uF, Capacitor_SMD:C_0805_2012Metric, F.Cu at (139.0, 110.5)
- added C3: 0.1uF, Capacitor_SMD:C_0805_2012Metric, F.Cu at (72.5, 79.3)
- added C30: 0.1uF, Capacitor_SMD:C_0805_2012Metric, F.Cu at (109.5, 168.0)
- added C31: 0.1uF, Capacitor_SMD:C_0805_2012Metric, F.Cu at (126.5, 157.5)
- added C32: 0.1uF, Capacitor_SMD:C_0805_2012Metric, F.Cu at (112.1, 151.6)
- added C33: 0.1uF, Capacitor_SMD:C_0805_2012Metric, F.Cu at (116.5, 151.6)
- added C34: 0.1uF, Capacitor_SMD:C_0805_2012Metric, F.Cu at (103.8, 103.3)
- added C35: 0.1uF, Capacitor_SMD:C_0805_2012Metric, F.Cu at (107.3, 103.3)
- added C36: 0.1uF, Capacitor_SMD:C_0805_2012Metric, F.Cu at (103.9, 113.1)
- added C37: 0.1uF, Capacitor_SMD:C_0805_2012Metric, F.Cu at (107.4, 113.1)
- added C4: 1000uF, Capacitor_SMD:CP_Elec_16x17.5, F.Cu at (102.5, 86.0)
- added C5: 22uF, Capacitor_SMD:C_0805_2012Metric, F.Cu at (119.0, 82.4)
- added C6: 0.01uF, Capacitor_SMD:C_0805_2012Metric, F.Cu at (51.0, 139.2)
- added C7: 1uF, Capacitor_SMD:C_0805_2012Metric, F.Cu at (53.2, 139.3)
- added C8: 470pF, Capacitor_SMD:C_0805_2012Metric, F.Cu at (59.7, 131.0)
- added C9: 0.1uF, Capacitor_SMD:C_0805_2012Metric, F.Cu at (73.5, 162.6)
- added D1: SSA33L, Diode_SMD:D_SMA, F.Cu at (62.0, 85.5)
- added D10: 1N4448, Diode_SMD:D_SOD-123, F.Cu at (59.8, 117.2)
- added D11: LED, LED_SMD:LED_0805_2012Metric, F.Cu at (56.8, 123.5)
- added D12: 1N4448, Diode_SMD:D_SOD-123, F.Cu at (59.8, 122.2)
- added D13: LED, LED_SMD:LED_0805_2012Metric, F.Cu at (76.7, 118.3)
- added D14: LED, LED_SMD:LED_0805_2012Metric, F.Cu at (76.5, 116.2)
- added D15: LED, LED_SMD:LED_0805_2012Metric, F.Cu at (76.7, 126.5)
- added D16: LED, LED_SMD:LED_0805_2012Metric, F.Cu at (76.7, 124.4)
- added D17: 1N4448, Diode_SMD:D_SOD-123, F.Cu at (79.5, 109.6)
- added D18: 1N4448, Diode_SMD:D_SOD-123, F.Cu at (79.5, 106.5)
- added D19: 1N4448, Diode_SMD:D_SOD-123, F.Cu at (79.5, 103.1)
- added D2: 50WQ04, Package_TO_SOT_SMD:TO-252-3_TabPin4, F.Cu at (81.8, 81.0)
- added D20: 1N4448, Diode_SMD:D_SOD-123, F.Cu at (79.5, 100.5)
- added D3: PZU5.1B2A, Diode_SMD:D_SOD-323, F.Cu at (80.6, 138.2)
- added D4: PZU5.1B2A, Diode_SMD:D_SOD-323, F.Cu at (57.2, 152.6)
- added D5: LED, LED_SMD:LED_0805_2012Metric, F.Cu at (56.8, 106.2)
- added D6: 1N4448, Diode_SMD:D_SOD-123, F.Cu at (59.8, 107.5)
- added D7: LED, LED_SMD:LED_0805_2012Metric, F.Cu at (56.8, 113.8)
- added D8: 1N4448, Diode_SMD:D_SOD-123, F.Cu at (59.8, 112.2)
- added D9: LED, LED_SMD:LED_0805_2012Metric, F.Cu at (56.8, 116.0)
- added F1: Polyfuse, Fuse:Fuse_1812_4532Metric, F.Cu at (95.5, 98.2)
- added F2: Polyfuse, Fuse:Fuse_1812_4532Metric, F.Cu at (144.0, 91.0)
- added G***: LOGO, LOGO, B.Cu at (84.7, 82.4)
- added H1: MountingHole, MountingHole:MountingHole_4.3mm_M4_Pad, F.Cu at (53.0, 171.2)
- added H2: MountingHole, MountingHole:MountingHole_4.3mm_M4_Pad, F.Cu at (53.0, 82.2)
- added H3: MountingHole, MountingHole:MountingHole_4.3mm_M4_Pad, F.Cu at (142.0, 82.2)
- added H4: MountingHole, MountingHole:MountingHole_4.3mm_M4_Pad, F.Cu at (142.0, 171.2)
- added IC1: Trig Cond Socket, Package_DIP:DIP-8_W7.62mm_Socket, F.Cu at (91.7, 161.7)
- added IC2: Trig Cond Socket, Package_DIP:DIP-8_W7.62mm_Socket, F.Cu at (91.8, 149.9)
- added J1: Conn_02x20_Odd_Even, Connector_IDC:IDC-Header_2x20_P2.54mm_Vertical, F.Cu at (65.2, 110.1)
- added J2: Conn_01x02, TerminalBlock_Phoenix:TerminalBlock_Phoenix_MKDS-1,5-2-5.08_1x02_P5.08mm_Horizontal, F.Cu at (52.6, 90.2)
- added J3: MAP_Connector, Connector_PinSocket_2.54mm:PinSocket_1x03_P2.54mm_Vertical, F.Cu at (52.0, 130.5)
- added J4: Conn_01x06, Connector_PinHeader_2.54mm:PinHeader_1x06_P2.54mm_Vertical, F.Cu at (143.9, 149.6)
- added J5: Conn_01x05, Connector_PinHeader_2.54mm:PinHeader_1x05_P2.54mm_Vertical, F.Cu at (144.0, 95.9)
- added J6: Conn_01x05, Connector_PinHeader_2.54mm:PinHeader_1x05_P2.54mm_Vertical, F.Cu at (143.9, 122.9)
- added J8: Conn_01x04, Connector_PinHeader_2.54mm:PinHeader_1x04_P2.54mm_Vertical, F.Cu at (144.0, 111.0)
- added JP1: MAP-SEL, Connector_PinHeader_2.54mm:PinHeader_1x03_P2.54mm_Vertical, F.Cu at (56.0, 135.5)
- added JP2: PULL-UP, Connector_PinHeader_2.54mm:PinHeader_1x02_P2.54mm_Vertical, F.Cu at (73.9, 153.6)
- added JP3: VR-HALL, Connector_PinHeader_2.54mm:PinHeader_1x03_P2.54mm_Vertical, F.Cu at (81.4, 153.6)
- added JP4: PULL-UP, Connector_PinHeader_2.54mm:PinHeader_1x02_P2.54mm_Vertical, F.Cu at (73.9, 157.3)
- added JP5: VR-HALL, Connector_PinHeader_2.54mm:PinHeader_1x03_P2.54mm_Vertical, F.Cu at (81.4, 157.3)
- added JP6: PULL-UP, Connector_PinHeader_2.54mm:PinHeader_1x02_P2.54mm_Vertical, F.Cu at (74.0, 149.8)
- added JP7: VR-HALL, Connector_PinHeader_2.54mm:PinHeader_1x03_P2.54mm_Vertical, F.Cu at (81.5, 149.8)
- added JP8: Ignition Voltage, Connector_PinHeader_2.54mm:PinHeader_1x03_P2.54mm_Vertical, F.Cu at (94.5, 123.8)
- added L1: 100uH, Inductor_SMD:L_12x12mm_H8mm, F.Cu at (84.8, 91.5)
- added Q1: SSM3K318R, Package_TO_SOT_SMD:SOT-23, F.Cu at (52.9, 151.6)
- added Q2: SSM3K318R, Package_TO_SOT_SMD:SOT-23, F.Cu at (52.8, 144.0)
- added Q3: SSM3K318R, Package_TO_SOT_SMD:SOT-23, F.Cu at (52.8, 147.8)
- added R0: 120R, Resistor_SMD:R_0603_1608Metric, F.Cu at (119.2, 80.5)
- added R1: 10kR, Resistor_SMD:R_0805_2012Metric, F.Cu at (133.0, 80.7)
- added R10: 2k49R +/-0.1%, Resistor_SMD:R_0805_2012Metric, F.Cu at (56.2, 156.1)
- added R11: 470R, Resistor_SMD:R_0805_2012Metric, F.Cu at (60.2, 156.2)
- added R12: 2k4R, Resistor_SMD:R_0805_2012Metric, F.Cu at (56.5, 141.2)
- added R13: 1kR, Resistor_SMD:R_0402_1005Metric, F.Cu at (60.0, 152.8)
- added R14: 1kR, Resistor_SMD:R_0402_1005Metric, F.Cu at (78.9, 154.1)
- added R15: 220R, Resistor_SMD:R_0603_1608Metric, F.Cu at (104.0, 160.8)
- added R16: 1kR, Resistor_SMD:R_0402_1005Metric, F.Cu at (78.9, 157.1)
- added R17: 220R, Resistor_SMD:R_0603_1608Metric, F.Cu at (104.0, 164.8)
- added R18: 1kR, Resistor_SMD:R_0402_1005Metric, F.Cu at (79.0, 149.3)
- added R19: 220R, Resistor_SMD:R_0603_1608Metric, F.Cu at (104.2, 151.0)
- added R2: 470R, Resistor_SMD:R_0805_2012Metric, F.Cu at (59.6, 133.0)
- added R20: 100kR, Resistor_SMD:R_0402_1005Metric, F.Cu at (49.5, 108.5)
- added R21: 1kR, Resistor_SMD:R_0402_1005Metric, F.Cu at (50.5, 108.5)
- added R22: 1kR, Resistor_SMD:R_0402_1005Metric, F.Cu at (50.5, 112.1)
- added R23: 100kR, Resistor_SMD:R_0402_1005Metric, F.Cu at (49.5, 112.1)
- added R24: 2k4R, Resistor_SMD:R_0805_2012Metric, F.Cu at (53.2, 106.2)
- added R25: 2k4R, Resistor_SMD:R_0805_2012Metric, F.Cu at (53.2, 113.8)
- added R26: 100kR, Resistor_SMD:R_0402_1005Metric, F.Cu at (49.5, 118.2)
- added R27: 1kR, Resistor_SMD:R_0402_1005Metric, F.Cu at (50.5, 118.2)
- added R28: 1kR, Resistor_SMD:R_0402_1005Metric, F.Cu at (50.5, 121.0)
- added R29: 100kR, Resistor_SMD:R_0402_1005Metric, F.Cu at (49.5, 121.0)
- added R3: 470R, Resistor_SMD:R_0805_2012Metric, F.Cu at (73.5, 160.6)
- added R30: 2k4R, Resistor_SMD:R_0805_2012Metric, F.Cu at (53.2, 116.0)
- added R31: 2k4R, Resistor_SMD:R_0805_2012Metric, F.Cu at (53.2, 123.5)
- added R32: 100kR, Resistor_SMD:R_0402_1005Metric, F.Cu at (91.2, 118.2)
- added R33: 1kR, Resistor_SMD:R_0402_1005Metric, F.Cu at (90.2, 118.2)
- added R34: 1kR, Resistor_SMD:R_0402_1005Metric, F.Cu at (90.2, 115.4)
- added R35: 100kR, Resistor_SMD:R_0402_1005Metric, F.Cu at (91.2, 115.4)
- added R36: 2k4R, Resistor_SMD:R_0805_2012Metric, F.Cu at (80.1, 118.2)
- added R37: 10R, Resistor_SMD:R_0402_1005Metric, F.Cu at (80.5, 119.7)
- added R38: 10R, Resistor_SMD:R_0402_1005Metric, F.Cu at (80.2, 114.7)
- added R39: 2k4R, Resistor_SMD:R_0805_2012Metric, F.Cu at (80.0, 116.2)
- added R4: 470R, Resistor_SMD:R_0805_2012Metric, F.Cu at (66.4, 167.1)
- added R40: 100kR, Resistor_SMD:R_0402_1005Metric, F.Cu at (91.2, 127.2)
- added R41: 1kR, Resistor_SMD:R_0402_1005Metric, F.Cu at (90.2, 127.2)
- added R42: 1kR, Resistor_SMD:R_0402_1005Metric, F.Cu at (90.2, 124.7)
- added R43: 100kR, Resistor_SMD:R_0402_1005Metric, F.Cu at (91.2, 124.7)
- added R44: 2k4R, Resistor_SMD:R_0805_2012Metric, F.Cu at (80.2, 126.5)
- added R45: 10R, Resistor_SMD:R_0402_1005Metric, F.Cu at (80.7, 128.0)
- added R46: 10R, Resistor_SMD:R_0402_1005Metric, F.Cu at (80.5, 122.9)
- added R47: 2k4R, Resistor_SMD:R_0805_2012Metric, F.Cu at (80.2, 124.4)
- added R48: 100kR, Resistor_SMD:R_0402_1005Metric, F.Cu at (91.0, 110.0)
- added R49: 1kR, Resistor_SMD:R_0402_1005Metric, F.Cu at (90.0, 110.0)
- added R5: 2k49R +/-0.1%, Resistor_SMD:R_0805_2012Metric, F.Cu at (61.6, 165.0)
- added R50: 1kR, Resistor_SMD:R_0402_1005Metric, F.Cu at (90.0, 107.5)
- added R51: 100kR, Resistor_SMD:R_0402_1005Metric, F.Cu at (91.0, 107.5)
- added R52: 100kR, Resistor_SMD:R_0402_1005Metric, F.Cu at (91.0, 104.2)
- added R53: 1kR, Resistor_SMD:R_0402_1005Metric, F.Cu at (90.0, 104.2)
- added R54: 1kR, Resistor_SMD:R_0402_1005Metric, F.Cu at (90.0, 101.5)
- added R55: 100kR, Resistor_SMD:R_0402_1005Metric, F.Cu at (91.0, 101.5)
- added R56: 10kR, Resistor_SMD:R_0805_2012Metric, F.Cu at (60.2, 149.8)
- added R57: 470R, Resistor_SMD:R_0805_2012Metric, F.Cu at (141.0, 110.5)
- added R58: 470R, Resistor_SMD:R_0805_2012Metric, F.Cu at (141.0, 114.0)
- added R6: 470R, Resistor_SMD:R_0805_2012Metric, F.Cu at (59.8, 163.0)
- added R60: 180kR +/-0.1%, Resistor_SMD:R_0805_2012Metric, F.Cu at (108.2, 164.2)
- added R61: 330kR +/-0.1%, Resistor_SMD:R_0805_2012Metric, F.Cu at (110.2, 164.2)
- added R62: 180kR +/-0.1%, Resistor_SMD:R_0805_2012Metric, F.Cu at (108.5, 171.2)
- added R63: 330kR +/-0.1%, Resistor_SMD:R_0805_2012Metric, F.Cu at (110.5, 171.2)
- added R64: 180kR +/-0.1%, Resistor_SMD:R_0805_2012Metric, F.Cu at (122.0, 169.2)
- added R65: 330kR +/-0.1%, Resistor_SMD:R_0805_2012Metric, F.Cu at (120.0, 169.2)
- added R66: 180kR +/-0.1%, Resistor_SMD:R_0805_2012Metric, F.Cu at (122.0, 164.0)
- added R67: 330kR +/-0.1%, Resistor_SMD:R_0805_2012Metric, F.Cu at (120.0, 164.0)
- added R68: 180kR +/-0.1%, Resistor_SMD:R_0805_2012Metric, F.Cu at (125.2, 154.7)
- added R69: 330kR +/-0.1%, Resistor_SMD:R_0805_2012Metric, F.Cu at (127.2, 154.8)
- added R7: 3k9R, Resistor_SMD:R_0805_2012Metric, F.Cu at (75.4, 135.2)
- added R70: 180kR +/-0.1%, Resistor_SMD:R_0805_2012Metric, F.Cu at (125.2, 160.3)
- added R71: 330kR +/-0.1%, Resistor_SMD:R_0805_2012Metric, F.Cu at (127.2, 160.3)
- added R8: 1kR, Resistor_SMD:R_0402_1005Metric, F.Cu at (75.4, 138.0)
- added R9: 470R, Resistor_SMD:R_0805_2012Metric, F.Cu at (80.6, 136.2)
- added RV1: Varistor, Capacitor_SMD:C_2220_5650Metric, F.Cu at (62.0, 80.5)
- added S1: MSS3-V-T_R, Speeduino-lib:MSS3VTR, F.Cu at (126.0, 83.7)
- added U1: Teensy4.1, Speeduino-lib:Teensy41, F.Cu at (124.5, 117.8)
- added U10: LM324A, Package_SO:SOIC-14_3.9x8.7mm_P1.27mm, F.Cu at (115.2, 166.5)
- added U11: LM324A, Package_SO:SOIC-14_3.9x8.7mm_P1.27mm, F.Cu at (132.0, 157.2)
- added U12: CD4504B, Package_SO:TSSOP-16_4.4x5mm_P0.65mm, F.Cu at (113.9, 155.5)
- added U13: CD4504B, Package_SO:TSSOP-16_4.4x5mm_P0.65mm, F.Cu at (105.6, 107.2)
- added U14: CD4504B, Package_SO:TSSOP-16_4.4x5mm_P0.65mm, F.Cu at (105.7, 117.0)
- added U2: LM2576-5G, Package_TO_SOT_SMD:TO-263-5_TabPin6, F.Cu at (67.5, 93.2)
- added U3: SP720, Package_SO:SOIC-16_3.9x9.9mm_P1.27mm, F.Cu at (83.2, 168.7)
- added U4: BM2LC105, Package_SO:SOP-8_3.9x4.9mm_P1.27mm, F.Cu at (54.8, 110.0)
- added U5: BM2LC105, Package_SO:SOP-8_3.9x4.9mm_P1.27mm, F.Cu at (54.8, 119.8)
- added U6: TC4424A, Package_SO:SOIC-8_3.9x4.9mm_P1.27mm, F.Cu at (85.7, 116.9)
- added U7: TC4424A, Package_SO:SOIC-8_3.9x4.9mm_P1.27mm, F.Cu at (85.7, 126.1)
- added U8: BM2LC105, Package_SO:SOP-8_3.9x4.9mm_P1.27mm, F.Cu at (85.7, 108.7)
- added U9: BM2LC105, Package_SO:SOP-8_3.9x4.9mm_P1.27mm, F.Cu at (85.7, 102.8)
Routing:
- net MAP-5V: track 0.00 -> 123.8 mm
- net FLEX-IN: track 0.00 -> 123.0 mm, vias 0 -> 2
- net MCU-FAN: track 0.00 -> 119.5 mm, vias 0 -> 1
- net MCU-PUMP: track 0.00 -> 113.7 mm, vias 0 -> 2
- net MCU-TACHO: track 0.00 -> 113.7 mm, vias 0 -> 3
- net MCU-ST-EN: track 0.00 -> 100.9 mm, vias 0 -> 2
- net CLT-5V: track 0.00 -> 99.3 mm, vias 0 -> 4
- net IAT-5V: track 0.00 -> 95.3 mm, vias 0 -> 2
- net CLUTCH-5V: track 0.00 -> 93.9 mm, vias 0 -> 2
- net GND: track 0.00 -> 92.9 mm, vias 0 -> 122
- net BAT-5V: track 0.00 -> 91.7 mm
- net MCU-ST-STEP: track 0.00 -> 91.1 mm, vias 0 -> 3
- net MCU-ST-DIR: track 0.00 -> 89.5 mm, vias 0 -> 2
- net INJ4-5V: track 0.00 -> 89.3 mm
- net INJ3-5V: track 0.00 -> 87.8 mm
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- added copper zone on F.Cu, net +12V
- added copper zone on In2.Cu, net +12V
- added copper zone on In2.Cu, net +3V3
- added copper zone on F.Cu, net GND
- added copper zone on In1.Cu, net GND
- added copper zone on B.Cu, net HC-1-OUT
- added copper zone on F.Cu, net HC-1-OUT
- added copper zone on B.Cu, net HC-2-OUT
- added copper zone on F.Cu, net HC-2-OUT
- added copper zone on B.Cu, net Net-(C1-Pad1)
- added copper zone on F.Cu, net Net-(C1-Pad1)
- added copper zone on F.Cu, net VDD
- added copper zone on In2.Cu, net VDD
- added copper zone on F.Cu, net VDDA
- added copper zone on In2.Cu, net VDDA
Other:
- board outline added: 100 x 100 mm
- board text added: "Fontys Engineering Eindhoven EXPO Group 13 Fall 2022"
